File: 12v driver/12v-driver.brd (EAGLE design)
At the start: 100 x 100 mm, 81 parts, among them IC1 74AC14D, IC3 4081N, IC4 74AC14D, Q1 BC618, Q11 BSS84, Q12 BSS84, Q13 2N2907, Q2 BC618, Q3 BC618, Q4 BC618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

Commit message: started routing v2
Parts:
- removed D1, D2, D3, D4: (no value), diode:DO-214AC
- removed IC3: 4081N, 40xx:DIL14
- removed Q10, Q9: (no value), adafruit:SOT23
- removed Q11, Q12: BSS84, Transistor:SOT23
- removed Q13: 2N2907, adafruit:TO92-EBC-OVAL
- removed T1: 2N2222, adafruit:TO92-EBC-OVAL
- added JP11, JP12, JP5, JP6: JUMPER-SMT_2_NO_NO-SILK, SparkFun-Jumpers:SMT-JUMPER_2_NO_NO-SILK
- added R26, R27: 10k, rcl:R0603
- added U$10, U$11, U$12, U$9: DSS110UTR, BLDC:SOD123FL
- added U$4: TC7PZ14FU,LJ(CT, BLDC:SOT-363___(US6)
- added U$5, U$6: SI2372DS-T1-GE3, BLDC:SOT-23
- added U$7, U$8: DMP2100U-7, BLDC:SOT-23
- added U1: SN74LVC2G08DCURDCU8-M, BLDC:DCU8-M
- Q1, Q2, Q3, Q4, Q5, Q6, Q7, Q8: value BC618 -> 2N3904; device transistor-npn:TO92-EBC -> BLDC:TO-92
- R10: value 2k -> 1k
- moved Q1 343.1 mm to (58.4, 87.6)
- moved Q3 336.6 mm to (58.4, 69.8)
- moved Q8 319.6 mm to (-49.5, 82.5)
- moved Q7 319.1 mm to (-41.9, 82.5)
- moved Q6 302.7 mm to (-95.2, 82.5)
- moved Q5 302.5 mm to (-87.6, 82.5)
- moved Q4 302.3 mm to (-80.0, 82.5)
- moved IC1 302.2 mm to (41.9, 69.8)
- moved Q2 301.9 mm to (-64.8, 82.5)
- moved C13 256.6 mm to (-101.6, 47.0)
- moved C14 256.6 mm to (-101.6, 43.2)
- moved C15 256.6 mm to (-101.6, 39.4)
- moved C16 256.6 mm to (-101.6, 35.6)
- moved D10 214.5 mm to (-63.5, 47.0)
- moved D11 214.5 mm to (-63.5, 35.6)
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Connections:
- removed net IN: Q13.B, T1.B
- removed net N$36: IC1.13, IC3.2
- removed net N$37: IC3.1, IC3.6
- removed net OUT: Q13.E, T1.E
- removed net VDD: IC3.14
- removed net VSS: IC3.7
- new net DIRECTION: R9.1, U$4.3, U1.2
- new net ENABLE: R10.1, U1.1, U1.6
- net +3V3: now also U$4.4, U1.8; no longer R10.1
- net GND: now also Q1.E, Q3.E, Q7.E, R10.2, R27.2, U$4.2, U$5.2, U$6.2, U1.4; no longer Q10.2, Q13.C, Q4.E, Q6.E, Q8.E, Q9.2
- net IN1: now also U1.3; no longer IC3.4, R9.1
- net IN2: now also U$4.6; no longer IC4.12, R10.2
- net N$1: now also R27.1
- net N$10: now also JP5.2, U$7.1; no longer Q12.1
- net N$11: now also JP5.1, U$6.1; no longer Q10.1
- net N$12: now also Q1.B; no longer Q2.B
- net N$13: now also U$10.A; no longer D4.A
- net N$15: now also U$4.5, U1.5; no longer IC1.12, IC3.5
- net N$16: now also U$10.C; no longer D4.C
- net N$18: now also U$12.A; no longer D1.A
- net N$20: now also U$11.C; no longer D2.C
- net N$22: now also U$11.A; no longer D2.A
- net N$23: now also U$12.C; no longer D1.C
- net N$25: now also U$9.C; no longer D3.C
- net N$26: now also U$9.A; no longer D3.A
- net N$3: now also Q3.C, Q4.B; no longer Q5.B, Q6.C
- net N$31: now also Q7.B; no longer Q8.B
- net N$32: now also Q7.C, Q8.B; no longer Q7.B, Q8.C
- net N$33: now also Q2.B; no longer Q4.B
- net N$35: now also Q2.C, Q5.B; no longer Q3.B, Q4.C
- net N$38: now also U$4.1, U1.7; no longer IC3.3, IC4.13
- net N$4: now also JP12.2, U$8.1; no longer Q11.1
- net N$40: now also U$7.3; no longer Q12.3
- net N$41: now also U$6.3; no longer Q10.3
- net N$42: now also U$5.3; no longer Q9.3
- net N$43: now also JP6.2, Q6.E; no longer Q1.E
- net N$44: now also JP6.1, Q5.E; no longer Q3.E
- net N$47: now also JP11.2, Q4.E; no longer Q5.E
- net N$48: now also JP11.1, Q8.E; no longer Q7.E
- net N$5: now also JP12.1, U$5.1
- net N$6: now also Q3.B; no longer Q6.B
- net N$7: now also R26.2
- net N$8: now also U$8.3; no longer Q11.3
- net N$9: now also Q1.C, Q6.B; no longer Q1.B, Q2.C
- net V+: now also Q4.C, Q6.C, Q8.C, R26.1, U$7.2, U$8.2; no longer Q1.C, Q11.2, Q12.2, Q3.C, Q7.C, T1.C
Routing:
- net N$34: track 31.9 -> 4.34 mm
- net N$28: track 28.4 -> 2.95 mm
- net N$21: track 28.0 -> 3.83 mm
- net ENABLE: track 0.00 -> 24.0 mm
- net N$17: track 25.9 -> 3.20 mm
- net IN2: track 35.9 -> 16.7 mm
- net IN1: track 37.9 -> 20.4 mm, vias 1 -> 0
- net DIRECTION: track 0.00 -> 16.1 mm
- net N$38: track 0.00 -> 10.6 mm
- net +3V3: track 2.32 -> 11.7 mm, vias 1 -> 3
- net N$27: track 8.64 -> 0.00 mm
- net N$15: track 0.00 -> 8.22 mm
- net N$13: track 2.70 -> 8.61 mm
- net N$14: track 2.66 -> 8.14 mm
- net N$20: track 13.1 -> 7.70 mm
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- added copper zone on layer 16, net +3V3
- removed copper zone on layer 16, net +5V

Commit message: made panel
Parts:
- removed C10, C5: (no value), rcl:C050-024X044
- removed C11, C12, C7, C8: (no value), rcl:C0603
- removed C6, C9: (no value), rcl:C075-032X103
- added C17, C18: (no value), rcl:C075-032X103
- added SV1: (no value), con-lstb:MA04-1
- added U2: V_REG_317SMD, SparkFun-IC-Power:SOT223
- moved JP12 214.4 mm to (69.6, 64.0), turned to 90 degrees
- moved JP11 204.2 mm to (67.6, 64.0), turned to 90 degrees
- moved JP6 202.9 mm to (66.8, 82.5), turned to 90 degrees
- moved JP5 196.6 mm to (68.6, 82.5), turned to 90 degrees
- moved D7 186.9 mm to (85.1, 78.7), turned to 90 degrees
- moved D8 183.3 mm to (86.4, 61.0), turned to 270 degrees
- moved R25 164.7 mm to (73.7, 63.5), turned to 180 degrees
- moved R22 164.4 mm to (71.1, 80.3), turned to 180 degrees
- moved R21 164.3 mm to (71.1, 85.1)
- moved R18 163.8 mm to (73.7, 65.3)
- moved C15 157.7 mm to (52.8, 71.4)
- moved Q6 157.7 mm to (62.2, 90.2), turned to 270 degrees
- moved C16 157.5 mm to (52.8, 66.3)
- moved C13 154.4 mm to (46.7, 89.7)
- moved C14 153.8 mm to (46.7, 83.8)
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Connections:
- new net N$36: SV1.1
- new net N$37: SV1.2
- new net N$46: SV1.3
- new net N$49: SV1.4
- net +3V3: now also C18.1, U2.2
- net GND: now also C17.2, C18.2, U2.1; no longer C10.2, C11.2, C12.2, C5.2, C6.2, C7.2, C8.2, C9.2
- net V+: now also C17.1, U2.3; no longer C10.1, C11.1, C12.1, C5.1, C6.1, C7.1, C8.1, C9.1
Routing:
- net N$7: track 7.22 -> 32.0 mm
- net OUTPUT: track 0.00 -> 16.0 mm
- net N$1: track 18.6 -> 4.27 mm
- net N$32: track 0.00 -> 14.2 mm
- net N$35: track 0.00 -> 13.5 mm
- net N$12: track 0.00 -> 11.4 mm
- net N$43: track 0.00 -> 10.8 mm
- net N$41: track 0.00 -> 10.5 mm
- net N$33: track 0.00 -> 10.4 mm
- net N$9: track 4.34 -> 14.7 mm
- net N$44: track 0.00 -> 10.3 mm
- net N$48: track 0.00 -> 10.3 mm
- net N$3: track 4.34 -> 14.2 mm
- net N$42: track 0.00 -> 9.42 mm
- net N$31: track 0.00 -> 8.77 mm
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