File: 12v driver/12v-driver.sch (EAGLE design)
At the start: 86 parts, among them IC1 74AC14D, IC4 74AC14D, Q1 2N3904, Q2 2N3904, Q3 2N3904, Q4 2N3904, Q5 2N3904, Q6 2N3904, Q7 2N3904, Q8 2N3904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

Commit message: made panel
Parts:
- removed C10, C5: (no value), rcl:C-US050-024X044
- removed C11, C12, C7, C8: (no value), rcl:C-USC0603
- removed C6, C9: (no value), rcl:C-US075-032X103
- added C17, C18: (no value), rcl:C-US075-032X103
- added SV1: (no value), con-lstb:MA04-1
- added U2: V_REG_317SMD, SparkFun-IC-Power:V_REG_317SMD
Connections:
- new net N$36: SV1.1
- new net N$37: SV1.2
- new net N$46: SV1.3
- new net N$49: SV1.4
- net +3V3: now also C18.1, U2.OUT
- net GND: now also C17.2, C18.2, U2.ADJ; no longer C10.2, C11.2, C12.2, C5.2, C6.2, C7.2, C8.2, C9.2
- net V+: now also C17.1, U2.IN; no longer C10.1, C11.1, C12.1, C5.1, C6.1, C7.1, C8.1, C9.1
