File: 12v driver/panel.sch (EAGLE design)
At the start: 79 parts, among them IC1 74AC14D, IC4 74AC14D, Q1 BC618, Q11 BSS84, Q12 BSS84, Q2 BC618, Q3 BC618, Q4 BC618, Q5 BC618, Q6 BC618, Q7 BC618, Q8 BC618, U1 SN74LVC2G08DCURDCU8-M

Commit message: made panel
Parts:
- removed C13, C14, C15, C16, C3, C4: (no value), rcl:C-USC0603
- removed D10, D11, D12, D7, D8, D9: (no value), diode:DIODE-DO-214AC
- removed D5, D6: WHITE, SparkFun-LED:LED-WHITE1206
- removed IC1, IC4: 74AC14D, 74xx-eu:74AC14D
- removed JP1, JP10, JP2, JP3, JP4, JP7, JP8, JP9: JUMPER-SMT_2_NO_NO-SILK, SparkFun-Jumpers:JUMPER-SMT_2_NO_NO-SILK
- removed Q1, Q2, Q3, Q4, Q5, Q6, Q7, Q8: BC618, transistor-npn:BC618
- removed R1, R11, R12, R19, R20, R4, R5, R8, R9: 1k, rcl:R-US_R0603
- removed R10, R13, R14, R15, R16, R17: 2k, rcl:R-US_R0603
- removed R18, R21, R22, R25: 30r, rcl:R-US_R0603
- removed R2, R3: 300r, rcl:R-US_R0603
- removed R23, R24: 10k, rcl:R-US_R0603
- removed R6, R7: 200r, rcl:R-US_R0603
- removed U$1: N-CHANNEL, transistors:N-CHANNEL
- removed U$2: P-CHANNEL, transistors:P-CHANNEL
- removed U$3: STM32F070F6P6TR, Capstone:STM32F070F6P6TR
- removed U1: SN74LVC2G08DCURDCU8-M, BLDC:SN74LVC2G08DCURDCU8-M
- added C31, C32, C33, C34, C35, C36, C37, C38, C51, C52, C53, C54, C55, C56, C57, C58: (no value), rcl:C-USC0603
- added D13, D14, D15, D16, D27, D28, D29, D30, D31, D32, D43, D44, D45, D46, D47, D48: (no value), diode:DIODE-DO-214AC
- added D25, D26, D41, D42: WHITE, SparkFun-LED:LED-WHITE1206
- added IC11, IC12, IC2, IC3, IC7, IC8: 74AC14D, 74xx-eu:74AC14D
- added JP13, JP14, JP15, JP16, JP17, JP18, JP19, JP20, JP21, JP22, JP23, JP24, JP37, JP38, JP39, JP40, JP41, JP42, JP43, JP44, JP45, JP46, JP47, JP48, JP61, JP62, JP63, JP64, JP65, JP66, JP67, JP68, JP69, JP70, JP71, JP72: JUMPER-SMT_2_NO_NO-SILK, SparkFun-Jumpers:JUMPER-SMT_2_NO_NO-SILK
- added Q13, Q14, Q15, Q16, Q25, Q26, Q27, Q28, Q29, Q30, Q31, Q32, Q41, Q42, Q43, Q44, Q45, Q46, Q47, Q48: 2N3904, BLDC:2N3904
- added R100, R106, R136, R139, R140, R143, R150, R151, R152, R153, R154, R160, R28, R31, R32, R35, R42, R43, R44, R45, R46, R52, R82, R85, R86, R89, R96, R97, R98, R99: 1k, rcl:R-US_R0603
- added R101, R102, R103, R104, R155, R156, R157, R158, R47, R48, R49, R50: 30r, rcl:R-US_R0603
- added R107, R108, R148, R149, R161, R162, R40, R41, R53, R54, R94, R95: 10k, rcl:R-US_R0603
- added R137, R138, R29, R30, R83, R84: 300r, rcl:R-US_R0603
- added R141, R142, R33, R34, R87, R88: 200r, rcl:R-US_R0603
- added R144, R145, R146, R147, R36, R37, R38, R39, R51, R90, R91, R92, R93: 2k, rcl:R-US_R0603
- added SV2: (no value), con-lstb:MA04-1
- added U$13, U$37, U$61: N-CHANNEL, transistors:N-CHANNEL
- added U$14, U$38, U$62: P-CHANNEL, transistors:P-CHANNEL
- added U$15: STM32F070F6P6TR, Capstone:STM32F070F6P6TR
- added U$16, U$40, U$64: TC7PZ14FU,LJ(CT, BLDC:TC7PZ14FU,LJ(CT
- added U$17, U$18, U$41, U$42, U$65, U$66: SI2372DS-T1-GE3, BLDC:SI2372DS-T1-GE3
- added U$19, U$20, U$43, U$44, U$67, U$68: DMP2100U-7, BLDC:DMP2100U-7
- added U$21, U$22, U$23, U$24, U$45, U$46, U$47, U$48, U$69, U$70, U$71, U$72: DSS110UTR, BLDC:DSS110UTR
- added U11, U3, U7: SN74LVC2G08DCURDCU8-M, BLDC:SN74LVC2G08DCURDCU8-M
- added U4: V_REG_317SMD, SparkFun-IC-Power:V_REG_317SMD
- C10, C5: device rcl:C-US050-024X044 -> rcl:C-USC0603
- C6, C9: device rcl:C-US075-032X103 -> rcl:C-USC0603
- D1, D2: value (none) -> WHITE; device diode:DIODE-DO-214AC -> SparkFun-LED:LED-WHITE1206
- Q10, Q9: value (none) -> 2N3904; device adafruit:MOSFET-NREFLOW -> BLDC:2N3904
- Q11, Q12: value BSS84 -> 2N3904; device Transistor:BSS84 -> BLDC:2N3904
Connections:
- removed net IN1: IC1B.I, IC1E.I, JP1.1, JP4.1, R9.1, U1G$2.O
- removed net IN2: IC4A.O, IC4B.I, IC4E.I, JP2.1, JP3.1, R10.2
- removed net N$1: R18.2, R25.1, U$1.G
- removed net N$10: Q12.G, R6.1
- removed net N$11: Q10.G, R7.1
- removed net N$12: C13.2, Q2.B, R8.1
- removed net N$13: D4.A, IC1B.O, R16.2
- removed net N$14: IC4C.O, JP7.1
- removed net N$15: IC1A.O, U1G$2.I0
- removed net N$16: C2.1, D4.C, IC1C.I, R16.1
- removed net N$17: C15.1, JP1.2, JP9.2, R4.2
- removed net N$18: C3.1, D1.A, IC4F.I, R14.1
- removed net N$19: IC4F.O, JP8.1
- removed net N$2: R17.2, U$3.BOOT0
- removed net N$20: C4.1, D2.C, IC4C.I, R13.1
- removed net N$21: C13.1, JP3.2, JP7.2, R8.2
- removed net N$22: D2.A, IC4B.O, R13.2
- removed net N$23: D1.C, IC4E.O, R14.2
- removed net N$24: IC1C.O, JP9.1
- removed net N$25: D3.C, IC1E.O, R15.2
- removed net N$26: C1.1, D3.A, IC1F.I, R15.1
- removed net N$27: IC1F.O, JP10.1
- removed net N$28: C16.1, JP10.2, JP4.2, R12.2
- removed net N$29: D5.A, R23.2
- removed net N$3: D11.C, Q5.B, Q6.C, R1.1
- removed net N$30: D6.A, R24.2
- removed net N$31: C16.2, Q8.B, R12.1
- removed net N$32: D12.C, Q7.B, Q8.C, R11.1
- removed net N$33: C14.2, Q4.B, R20.1
- removed net N$34: C14.1, JP2.2, JP8.2, R20.2
- removed net N$35: D10.C, Q3.B, Q4.C, R19.1
- removed net N$36: IC1A.I, U1G$1.I1
- removed net N$37: U1G$1.I0, U1G$2.I1
- removed net N$38: IC4A.I, U1G$1.O
- removed net N$4: Q11.G, R2.1
- removed net N$40: Q12.D, R21.1
- removed net N$41: D5.C, Q10.D, R22.2
- removed net N$42: Q9.D, R25.2
- removed net N$43: D9.A, Q1.E, R6.2
- removed net N$44: D10.A, Q3.E, R7.2
- removed net N$47: D11.A, Q5.E, R2.2
- removed net N$48: D12.A, Q7.E, R3.2
- removed net N$5: R3.1
- removed net N$6: C15.2, Q6.B, R4.1
- removed net N$7: R21.2, R22.1, U$2.G
- removed net N$8: Q11.D, R18.1, R24.1
- removed net N$9: D9.C, Q1.B, Q2.C, R5.1
- removed net OUTPUT: D7.A, D8.C, U$1.D, U$2.D
- removed net PWM1: U$3.PB1
- removed net PWM2: U$3.PA7
- removed net PWM3: U$3.PA6
- new net DIRECTION1: R42.1, U$15.PB1, U$16G$2.I, U3G$1.I1
- new net DIRECTION2: R96.1, U$15.PA7, U$40G$2.I, U7G$1.I1
- new net DIRECTION3: R150.1, U$15.PA6, U$64G$2.I, U11G$1.I1
- new net IN11: IC12B.I, IC12E.I, JP61.1, JP64.1, U11G$2.O
- new net IN12: IC11B.I, IC11E.I, JP62.1, JP63.1, U$64G$1.O
- new net IN3: IC3B.I, IC3E.I, JP13.1, JP16.1, U3G$2.O
- new net IN4: IC2B.I, IC2E.I, JP14.1, JP15.1, U$16G$1.O
- new net IN7: IC8B.I, IC8E.I, JP37.1, JP40.1, U7G$2.O
- new net IN8: IC7B.I, IC7E.I, JP38.1, JP39.1, U$40G$1.O
- new net N$145: R103.2, R104.1, R108.1, U$37.G
- new net N$146: JP48.2, R83.1, U$44.G
- new net N$147: JP48.1, R84.1, U$41.G
- new net N$148: C37.2, Q29.B, R85.1
- new net N$149: R101.2, R102.1, R107.2, U$38.G
- new net N$150: JP45.2, R87.1, U$43.G
- new net N$151: JP45.1, R88.1, U$42.G
- new net N$152: C35.2, Q27.B, R89.1
- new net N$153: C32.1, IC8C.I, R93.1, U$46.C
- new net N$154: C37.1, JP37.2, JP43.2, R85.2
- new net N$155: C33.1, IC7F.I, R91.1, U$48.A
- new net N$156: C34.1, IC7C.I, R90.1, U$47.C
- new net N$157: C35.1, JP39.2, JP41.2, R89.2
- new net N$158: IC7B.O, R90.2, U$47.A
- new net N$159: IC7E.O, R91.2, U$48.C
- new net N$160: IC8E.O, R92.2, U$45.C
- new net N$161: IC8B.O, R93.2, U$46.A
- new net N$162: D31.C, Q29.C, Q30.B, R82.1
- new net N$163: D29.C, Q27.C, Q32.B, R86.1
- new net N$164: C38.1, JP40.2, JP44.2, R98.2
- new net N$165: C31.1, IC8F.I, R92.1, U$45.A
- new net N$166: D25.A, R94.2
- new net N$167: D26.A, R95.2
- new net N$168: IC7C.O, JP41.1
- new net N$169: IC7F.O, JP42.1
- new net N$170: IC8C.O, JP43.1
- new net N$171: IC8F.O, JP44.1
- new net N$172: C38.2, Q25.B, R98.1
- new net N$173: D32.C, Q25.C, Q26.B, R97.1
- new net N$174: C36.2, Q28.B, R100.1
- new net N$175: C36.1, JP38.2, JP42.2, R100.2
- new net N$176: D30.C, Q28.C, Q31.B, R99.1
- new net N$177: U$40G$2.O, U7G$2.I0
- new net N$178: U$40G$1.I, U7G$1.O
- new net N$179: R101.1, U$43.D
- new net N$180: D25.C, R102.2, U$42.D
- new net N$181: R103.1, R95.1, U$44.D
- new net N$182: R104.2, U$41.D
- new net N$184: D29.A, JP46.2, Q32.E, R87.2
- new net N$185: D30.A, JP46.1, Q31.E, R88.2
- new net N$186: D31.A, JP47.2, Q30.E, R83.2
- new net N$187: D32.A, JP47.1, Q26.E, R84.2
- new net N$241: R157.2, R158.1, R162.1, U$61.G
- new net N$242: JP72.2, R137.1, U$68.G
- new net N$243: JP72.1, R138.1, U$65.G
- new net N$244: C57.2, Q45.B, R139.1
- new net N$245: R155.2, R156.1, R161.2, U$62.G
- new net N$246: JP69.2, R141.1, U$67.G
- new net N$247: JP69.1, R142.1, U$66.G
- new net N$248: C55.2, Q43.B, R143.1
- new net N$249: C52.1, IC12C.I, R147.1, U$70.C
- new net N$250: C57.1, JP61.2, JP67.2, R139.2
- new net N$251: C53.1, IC11F.I, R145.1, U$72.A
- new net N$252: C54.1, IC11C.I, R144.1, U$71.C
- new net N$253: C55.1, JP63.2, JP65.2, R143.2
- new net N$254: IC11B.O, R144.2, U$71.A
- new net N$255: IC11E.O, R145.2, U$72.C
- new net N$256: IC12E.O, R146.2, U$69.C
- new net N$257: IC12B.O, R147.2, U$70.A
- new net N$258: D47.C, Q45.C, Q46.B, R136.1
- new net N$259: D45.C, Q43.C, Q48.B, R140.1
- new net N$260: C58.1, JP64.2, JP68.2, R152.2
- new net N$261: C51.1, IC12F.I, R146.1, U$69.A
- new net N$262: D41.A, R148.2
- new net N$263: D42.A, R149.2
- new net N$264: IC11C.O, JP65.1
- new net N$265: IC11F.O, JP66.1
- new net N$266: IC12C.O, JP67.1
- new net N$267: IC12F.O, JP68.1
- new net N$268: C58.2, Q41.B, R152.1
- new net N$269: D48.C, Q41.C, Q42.B, R151.1
- new net N$270: C56.2, Q44.B, R154.1
- new net N$271: C56.1, JP62.2, JP66.2, R154.2
- new net N$272: D46.C, Q44.C, Q47.B, R153.1
- new net N$273: U$64G$2.O, U11G$2.I0
- new net N$274: U$64G$1.I, U11G$1.O
- new net N$275: R155.1, U$67.D
- new net N$276: D41.C, R156.2, U$66.D
- new net N$277: R149.1, R157.1, U$68.D
- new net N$278: R158.2, U$65.D
- new net N$280: D45.A, JP70.2, Q48.E, R141.2
- new net N$281: D46.A, JP70.1, Q47.E, R142.2
- new net N$282: D47.A, JP71.2, Q46.E, R137.2
- new net N$283: D48.A, JP71.1, Q42.E, R138.2
- new net N$50: JP24.2, R29.1, U$20.G
- new net N$51: JP24.1, R30.1, U$17.G
- new net N$52: C11.2, Q13.B, R31.1
- new net N$53: R47.2, R48.1, R53.2, U$14.G
- new net N$54: JP21.2, R33.1, U$19.G
- new net N$55: JP21.1, R34.1, U$18.G
- new net N$56: C9.2, Q11.B, R35.1
- new net N$57: C6.1, IC3C.I, R39.1, U$22.C
- new net N$58: C11.1, JP13.2, JP19.2, R31.2
- new net N$59: C7.1, IC2F.I, R37.1, U$24.A
- new net N$60: C8.1, IC2C.I, R36.1, U$23.C
- new net N$61: C9.1, JP15.2, JP17.2, R35.2
- new net N$62: IC2B.O, R36.2, U$23.A
- new net N$63: IC2E.O, R37.2, U$24.C
- new net N$64: IC3E.O, R38.2, U$21.C
- new net N$65: IC3B.O, R39.2, U$22.A
- new net N$66: D15.C, Q13.C, Q14.B, R28.1
- new net N$67: D13.C, Q11.C, Q16.B, R32.1
- new net N$68: C12.1, JP16.2, JP20.2, R44.2
- new net N$69: C5.1, IC3F.I, R38.1, U$21.A
- new net N$70: D1.A, R40.2
- new net N$71: D2.A, R41.2
- new net N$72: IC2C.O, JP17.1
- new net N$73: IC2F.O, JP18.1
- new net N$74: IC3C.O, JP19.1
- new net N$75: IC3F.O, JP20.1
- new net N$76: C12.2, Q9.B, R44.1
- new net N$77: D16.C, Q10.B, Q9.C, R43.1
- new net N$78: C10.2, Q12.B, R46.1
- new net N$79: C10.1, JP14.2, JP18.2, R46.2
- new net N$80: D14.C, Q12.C, Q15.B, R45.1
- new net N$81: U$16G$2.O, U3G$2.I0
- new net N$82: U$16G$1.I, U3G$1.O
- new net N$83: R47.1, U$19.D
- new net N$84: D1.C, R48.2, U$18.D
- new net N$85: R41.1, R49.1, U$20.D
- new net N$86: R50.2, U$17.D
- new net N$87: R51.2, U$15.BOOT0
- new net N$88: D13.A, JP22.2, Q16.E, R33.2
- new net N$89: D14.A, JP22.1, Q15.E, R34.2
- new net N$90: D15.A, JP23.2, Q14.E, R29.2
- new net N$91: D16.A, JP23.1, Q10.E, R30.2
- new net N$93: SV2.1
- new net N$94: SV2.2
- new net N$95: SV2.3
- new net N$96: SV2.4
- new net OUTPUT1: D3.A, D4.C, U$13.D, U$14.D
- new net OUTPUT2: D27.A, D28.C, U$37.D, U$38.D
- new net OUTPUT3: D43.A, D44.C, U$61.D, U$62.D
- net +3V3: now also C2.1, IC11P.VCC, IC12P.VCC, IC2P.VCC, IC3P.VCC, IC7P.VCC, IC8P.VCC, U$15.VDD, U$15.VDDA, U$16G$3.VCC, U$40G$3.VCC, U$64G$3.VCC, U11G$3.VCC, U3G$3.VCC, U4.OUT, U7G$3.VCC; no longer IC1P.VCC, R10.1, U$3.VDD, U$3.VDDA, U1G$3.VCC
- net ADC1: now also U$15.PA0; no longer U$3.PA0
- net ADC2: now also U$15.PA1; no longer U$3.PA1
- net ADC3: now also U$15.PA2; no longer U$3.PA2
- net ENABLE1: now also R52.1, U$15.PA10, U3G$1.I0, U3G$2.I1; no longer U$3.PA10
- net ENABLE2: now also R106.1, U$15.PA9, U7G$1.I0, U7G$2.I1; no longer U$3.PA9
- net ENABLE3: now also R160.1, U$15.PA5, U11G$1.I0, U11G$2.I1; no longer U$3.PA5
- net GND: now also C31.2, C32.2, C33.2, C34.2, C51.2, C52.2, C53.2, C54.2, D2.C, D26.C, D28.A, D4.A, D42.C, D44.A, IC11P.GND, IC12P.GND, IC2P.GND, IC3P.GND, IC7P.GND, IC8P.GND, Q11.E, Q12.E, Q13.E, Q25.E, Q27.E, Q28.E, Q29.E, Q41.E, Q43.E, Q44.E, Q45.E, Q9.E, R106.2, R108.2, R150.2, R160.2, R162.2, R42.2, R51.1, R52.2, R54.2, R96.2, U$13.S, U$15.VSS, U$16G$3.GND, U$17.S, U$18.S, U$37.S, U$40G$3.GND, U$41.S, U$42.S, U$61.S, U$64G$3.GND, U$65.S, U$66.S, U11G$3.GND, U3G$3.GND, U4.ADJ, U7G$3.GND; no longer C10.2, C11.2, C12.2, C3.2, C4.2, C9.2, D6.C, D8.A, IC1P.GND, Q10.S, Q2.E, Q4.E, Q6.E, Q8.E, Q9.S, R17.1, R9.2, U$1.S, U$3.VSS, U1G$3.GND
- net HALF_VCC: now also U$15.PA3; no longer U$3.PA3
- net N$39: now also R49.2, R50.1, R54.1, U$13.G, U$15.NRST; no longer U$3.NRST
- net SWCLK: now also U$15.PA14; no longer U$3.PA14
- net SWDIO: now also U$15.PA13; no longer U$3.PA13
- net V+: now also C1.1, D27.C, D3.C, D43.C, Q10.C, Q14.C, Q15.C, Q16.C, Q26.C, Q30.C, Q31.C, Q32.C, Q42.C, Q46.C, Q47.C, Q48.C, R107.1, R136.2, R140.2, R148.1, R151.2, R153.2, R161.1, R28.2, R32.2, R40.1, R43.2, R45.2, R53.1, R82.2, R86.2, R94.1, R97.2, R99.2, U$14.S, U$19.S, U$20.S, U$38.S, U$43.S, U$44.S, U$62.S, U$67.S, U$68.S, U4.IN; no longer C10.1, C11.1, C12.1, C5.1, C6.1, C7.1, C8.1, C9.1, D7.C, Q1.C, Q11.S, Q12.S, Q3.C, Q5.C, Q7.C, R1.2, R11.2, R19.2, R23.1, R5.2, U$2.S
Other:
- moved on the sheet: C1, C10, C11, C12, C2, C5, C6, C7, C8, C9, D3, D4
